File: hw/saber/saber.kicad_pcb (KiCad board)
At the start: 2 copper layers, 2 parts, among them Q6 PSMN3R0-30MLC,115, U3 STM32L031F4Px

Commit message: better hierarchy; more footprint assignment
Parts:
- removed Q6: PSMN3R0-30MLC,115, Package_TO_SOT_SMD:LFPAK33
- removed U3: STM32L031F4Px, Package_SO:TSSOP-20_4.4x6.5mm_P0.65mm
Routing:
- removed copper zone on F.Cu, net GND
Changed lines of the file:
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@@
     (tracks 0)
     (zones 0)
-    (modules 2)
-    (nets 21)
+    (modules 0)
+    (nets 1)
   )
   (page A4)
@@
   )
   (net 0 "")
-  (net 1 /actuators/SIG_SOL)
-  (net 2 GND)
-  (net 3 /SOL-)
-  (net 4 /micro/BOOT0)
-  (net 5 /actuators/SIG_LED)
-  (net 6 /micro/NRST)
-  (net 7 +3V3)
-  (net 8 /micro/imtr)
-  (net 9 /micro/PWM_MTR)
-  (net 10 /micro/INA)
-  (net 11 /micro/INB)
-  (net 12 /micro/ADC_VBATT)
-  (net 13 /actuators/PWM_SPKR)
-  (net 14 "Net-(U3-Pad12)")
-  (net 15 /micro/LED_HBEAT)
-  (net 16 /micro/BTN)
-  (net 17 /micro/SCL)
-  (net 18 /micro/SDA)
-  (net 19 /micro/SWDIO)
-  (net 20 /micro/SWCLK)
   (net_class Default "This is the default net class."
     (clearance 0.2)
@@
     (uvia_dia 0.3)
     (uvia_drill 0.1)
-    (add_net +3V3)
-    (add_net /SOL-)
-    (add_net /actuators/PWM_SPKR)
-    (add_net /actuators/SIG_LED)
-    (add_net /actuators/SIG_SOL)
-    (add_net /micro/ADC_VBATT)
-    (add_net /micro/BOOT0)
-    (add_net /micro/BTN)
-    (add_net /micro/INA)
-    (add_net /micro/INB)
-    (add_net /micro/LED_HBEAT)
-    (add_net /micro/NRST)
-    (add_net /micro/PWM_MTR)
-    (add_net /micro/SCL)
-    (add_net /micro/SDA)
-    (add_net /micro/SWCLK)
-    (add_net /micro/SWDIO)
-    (add_net /micro/imtr)
-    (add_net GND)
-    (add_net "Net-(U3-Pad12)")
-  )
-  (module Package_TO_SOT_SMD:LFPAK33 (layer F.Cu)
-    (at 266.265001 52.725001)
-    (descr "LFPAK33 SOT-1210 https://assets.nexperia.com/documents/outline-drawing/SOT1210.pdf")
-    (tags "LFPAK33 SOT-1210")
-    (solder_mask_margin 0.05)
-    (attr smd)
-    (fp_text reference Q6 (at 0 -2.55) (layer F.SilkS)
-      (effects (font (size 1 1) (thickness 0.15)))
-    )
-    (fp_text value PSMN3R0-30MLC,115 (at 0 2.64) (layer F.Fab)
-      (effects (font (size 1 1) (thickness 0.15)))
-    )
-    (fp_text user %R (at 0 0 90) (layer F.Fab)
-      (effects (font (size 0.75 0.75) (thickness 0.13)))
-    )
-    (fp_line (start -1.22 1.475) (end -1.22 1.77) (layer F.SilkS) (width 0.12))
-    (fp_line (start -1.22 1.77) (end 1.62 1.77) (layer F.SilkS) (width 0.12))
-    (fp_line (start 1.62 1.77) (end 1.62 1.475) (layer F.SilkS) (width 0.12))
-    (fp_line (start 1.62 -1.475) (end 1.62 -1.77) (layer F.SilkS) (width 0.12))
-    (fp_line (start 1.62 -1.77) (end -1.22 -1.77) (layer F.SilkS) (width 0.12))
-    (fp_line (start -1.22 -1.77) (end -1.22 -1.475) (layer F.SilkS) (width 0.12))
-    (fp_line (start -0.6 -1.65) (end 1.5 -1.65) (layer F.Fab) (width 0.1))
-    (fp_line (start -1.1 -1.15) (end -1.1 1.65) (layer F.Fab) (width 0.1))
-    (fp_line (start -1.1 1.65) (end 1.5 1.65) (layer F.Fab) (width 0.1))
-    (fp_line (start 1.5 1.65) (end 1.5 -1.65) (layer F.Fab) (width 0.1))
-    (fp_line (start 2.2 -1.9) (end 2.2 1.9) (layer F.CrtYd) (width 0.05))
-    (fp_line (start -2.2 -1.9) (end 2.2 -1.9) (layer F.CrtYd) (width 0.05))
-    (fp_line (start -2.2 1.9) (end 2.2 1.9) (layer F.CrtYd) (width 0.05))
-    (fp_line (start -2.2 1.9) (end -2.2 -1.9) (layer F.CrtYd) (width 0.05))
-    (fp_line (start -1.95 -1.475) (end -1.22 -1.475) (layer F.SilkS) (width 0.12))
-    (fp_line (start -0.6 -1.65) (end -1.1 -1.15) (layer F.Fab) (width 0.1))
-    (pad "" smd rect (at -0.215 -0.626) (size 0.51 0.635) (layers F.Paste))
-    (pad "" smd rect (at 0.645 -0.626) (size 0.51 0.635) (layers F.Paste))
-    (pad "" smd rect (at -0.215 0.626) (size 0.51 0.635) (layers F.Paste))
-    (pad "" smd rect (at 0.645 0.626) (size 0.51 0.635) (layers F.Paste))
-    (pad 1 smd rect (at 1.575 -0.975) (size 0.75 0.4) (layers F.Cu F.Mask)
-      (net 2 GND))
-    (pad 1 smd rect (at 1.575 0.975) (size 0.75 0.4) (layers F.Cu F.Mask)
-      (net 2 GND))
-    (pad 1 smd rect (at 1.575 -0.325) (size 0.75 0.4) (layers F.Cu F.Mask)
-      (net 2 GND))
-    (pad 2 smd rect (at -1.535 -0.325) (size 0.83 0.4) (layers F.Cu F.Mask)
-      (net 1 /actuators/SIG_SOL))
-    (pad 1 smd rect (at -1.535 -0.975) (size 0.83 0.4) (layers F.Cu F.Mask)
-      (net 2 GND))
-    (pad 3 smd rect (at -1.535 0.325) (size 0.83 0.4) (layers F.Cu F.Mask)
-      (net 3 /SOL-))
-    (pad 1 smd rect (at 0.405 0) (size 1.85 2.25) (layers F.Cu F.Mask)
-      (net 2 GND))
-    (pad "" smd rect (at -1.535 0.975) (size 0.83 0.3) (layers F.Paste))
-    (pad 1 smd rect (at 1.575 0.325) (size 0.75 0.4) (layers F.Cu F.Mask)
-      (net 2 GND))
-    (pad 4 smd rect (at -1.535 0.975) (size 0.83 0.4) (layers F.Cu F.Mask))
-    (pad "" smd rect (at -1.535 0.325) (size 0.83 0.3) (layers F.Paste))
-    (pad "" smd rect (at -1.535 -0.325) (size 0.83 0.3) (layers F.Paste))
-    (pad "" smd rect (at -1.535 -0.975) (size 0.83 0.3) (layers F.Paste))
-    (pad "" smd rect (at 1.575 -0.975) (size 0.75 0.3) (layers F.Paste))
-    (pad "" smd rect (at 1.575 -0.325) (size 0.75 0.3) (layers F.Paste))
-    (pad "" smd rect (at 1.575 0.325) (size 0.75 0.3) (layers F.Paste))
-    (pad "" smd rect (at 1.575 0.975) (size 0.75 0.3) (layers F.Paste))
-    (model ${KISYS3DMOD}/Package_TO_SOT_SMD.3dshapes/LFPAK33.wrl
-      (at (xyz 0 0 0))
-      (scale (xyz 1 1 1))
-      (rotate (xyz 0 0 0))
-    )
-  )
-  (module Package_SO:TSSOP-20_4.4x6.5mm_P0.65mm (layer F.Cu)
-    (at 251.625001 54.375001)
-    (descr "20-Lead Plastic Thin Shrink Small Outline (ST)-4.4 mm Body [TSSOP] (see Microchip Packaging Specification 00000049BS.pdf)")
-    (tags "SSOP 0.65")
-    (attr smd)
-    (fp_text reference U3 (at 0 -4.3) (layer F.SilkS)
-      (effects (font (size 1 1) (thickness 0.15)))
-    )
-    (fp_text value STM32L031F4Px (at 0 4.3) (layer F.Fab)
-      (effects (font (size 1 1) (thickness 0.15)))
-    )
-    (fp_line (start -1.2 -3.25) (end 2.2 -3.25) (layer F.Fab) (width 0.15))
-    (fp_line (start 2.2 -3.25) (end 2.2 3.25) (layer F.Fab) (width 0.15))
-    (fp_line (start 2.2 3.25) (end -2.2 3.25) (layer F.Fab) (width 0.15))
-    (fp_line (start -2.2 3.25) (end -2.2 -2.25) (layer F.Fab) (width 0.15))
-    (fp_line (start -2.2 -2.25) (end -1.2 -3.25) (layer F.Fab) (width 0.15))
-    (fp_line (start -3.95 -3.55) (end -3.95 3.55) (layer F.CrtYd) (width 0.05))
-    (fp_line (start 3.95 -3.55) (end 3.95 3.55) (layer F.CrtYd) (width 0.05))
-    (fp_line (start -3.95 -3.55) (end 3.95 -3.55) (layer F.CrtYd) (width 0.05))
-    (fp_line (start -3.95 3.55) (end 3.95 3.55) (layer F.CrtYd) (width 0.05))
-    (fp_line (start -2.225 3.45) (end 2.225 3.45) (layer F.SilkS) (width 0.15))
-    (fp_line (start -3.75 -3.45) (end 2.225 -3.45) (layer F.SilkS) (width 0.15))
-    (fp_text user %R (at 0 0) (layer F.Fab)
-      (effects (font (size 0.8 0.8) (thickness 0.15)))
-    )
-    (pad 1 smd rect (at -2.95 -2.925) (size 1.45 0.45) (layers F.Cu F.Paste F.Mask)
-      (net 4 /micro/BOOT0))
-    (pad 2 smd rect (at -2.95 -2.275) (size 1.45 0.45) (layers F.Cu F.Paste F.Mask)
-      (net 5 /actuators/SIG_LED))
-    (pad 3 smd rect (at -2.95 -1.625) (size 1.45 0.45) (layers F.Cu F.Paste F.Mask)
-      (net 1 /actuators/SIG_SOL))
-    (pad 4 smd rect (at -2.95 -0.975) (size 1.45 0.45) (layers F.Cu F.Paste F.Mask)
-      (net 6 /micro/NRST))
-    (pad 5 smd rect (at -2.95 -0.325) (size 1.45 0.45) (layers F.Cu F.Paste F.Mask)
-      (net 7 +3V3))
-    (pad 6 smd rect (at -2.95 0.325) (size 1.45 0.45) (layers F.Cu F.Paste F.Mask)
-      (net 8 /micro/imtr))
-    (pad 7 smd rect (at -2.95 0.975) (size 1.45 0.45) (layers F.Cu F.Paste F.Mask)
-      (net 9 /micro/PWM_MTR))
-    (pad 8 smd rect (at -2.95 1.625) (size 1.45 0.45) (layers F.Cu F.Paste F.Mask)
-      (net 10 /micro/INA))
-    (pad 9 smd rect (at -2.95 2.275) (size 1.45 0.45) (layers F.Cu F.Paste F.Mask)
-      (net 11 /micro/INB))
-    (pad 10 smd rect (at -2.95 2.925) (size 1.45 0.45) (layers F.Cu F.Paste F.Mask)
-      (net 12 /micro/ADC_VBATT))
-    (pad 11 smd rect (at 2.95 2.925) (size 1.45 0.45) (layers F.Cu F.Paste F.Mask)
-      (net 13 /actuators/PWM_SPKR))
-    (pad 12 smd rect (at 2.95 2.275) (size 1.45 0.45) (layers F.Cu F.Paste F.Mask)
-      (net 14 "Net-(U3-Pad12)"))
-    (pad 13 smd rect (at 2.95 1.625) (size 1.45 0.45) (layers F.Cu F.Paste F.Mask)
-      (net 15 /micro/LED_HBEAT))
-    (pad 14 smd rect (at 2.95 0.975) (size 1.45 0.45) (layers F.Cu F.Paste F.Mask)
-      (net 16 /micro/BTN))
-    (pad 15 smd rect (at 2.95 0.325) (size 1.45 0.45) (layers F.Cu F.Paste F.Mask)
-      (net 2 GND))
-    (pad 16 smd rect (at 2.95 -0.325) (size 1.45 0.45) (layers F.Cu F.Paste F.Mask)
-      (net 7 +3V3))
-    (pad 17 smd rect (at 2.95 -0.975) (size 1.45 0.45) (layers F.Cu F.Paste F.Mask)
-      (net 17 /micro/SCL))
-    (pad 18 smd rect (at 2.95 -1.625) (size 1.45 0.45) (layers F.Cu F.Paste F.Mask)
-      (net 18 /micro/SDA))
-    (pad 19 smd rect (at 2.95 -2.275) (size 1.45 0.45) (layers F.Cu F.Paste F.Mask)
-      (net 19 /micro/SWDIO))
-    (pad 20 smd rect (at 2.95 -2.925) (size 1.45 0.45) (layers F.Cu F.Paste F.Mask)
-      (net 20 /micro/SWCLK))
-    (model ${KISYS3DMOD}/Package_SO.3dshapes/TSSOP-20_4.4x6.5mm_P0.65mm.wrl
-      (at (xyz 0 0 0))
-      (scale (xyz 1 1 1))
-      (rotate (xyz 0 0 0))
-    )
-  )
-  (zone (net 2) (net_name GND) (layer F.Cu) (hatch edge 0.508)
-    (connect_pads (clearance 0.508))
-    (min_thickness 0.254)
-    (fill yes (arc_segments 16) (thermal_gap 0.508) (thermal_bridge_width 0.508))
-    (polygon
-      (pts
-        (xy 263.525 50.165) (xy 268.605 50.165) (xy 268.605 53.34) (xy 263.525 51.435)
-      )
-    )
   )
 )

Commit message: reselected diodes, split up connector TBs for layout purposes
Parts:
- added C1: 33n, Capacitor_SMD:C_0603_1608Metric_Pad1.05x0.95mm_HandSolder, F.Cu at (66.1, 59.2)
- added C10: 470u, Capacitor_SMD:CP_Elec_16x17.5, F.Cu at (43.2, 77.5)
- added C11: 100n, Capacitor_SMD:C_0603_1608Metric_Pad1.05x0.95mm_HandSolder, F.Cu at (31.2, 47.5)
- added C12: 10u, Capacitor_SMD:C_0603_1608Metric_Pad1.05x0.95mm_HandSolder, F.Cu at (75.0, 56.0)
- added C13: 22u, Capacitor_SMD:C_0603_1608Metric_Pad1.05x0.95mm_HandSolder, F.Cu at (71.6, 57.6)
- added C14: 100n, Capacitor_SMD:C_0603_1608Metric_Pad1.05x0.95mm_HandSolder, F.Cu at (105.1, 38.6)
- added C15: 100n, Capacitor_SMD:C_0603_1608Metric_Pad1.05x0.95mm_HandSolder, F.Cu at (109.4, 34.4)
- added C16: 100n, Capacitor_SMD:C_0603_1608Metric_Pad1.05x0.95mm_HandSolder, F.Cu at (108.5, 38.6)
- added C17: 4u7, Capacitor_SMD:C_0603_1608Metric_Pad1.05x0.95mm_HandSolder, F.Cu at (109.4, 35.9)
- added C2: 100n, Capacitor_SMD:C_0603_1608Metric_Pad1.05x0.95mm_HandSolder, F.Cu at (85.3, 28.9)
- added C3: 10u, Capacitor_SMD:C_0603_1608Metric_Pad1.05x0.95mm_HandSolder, F.Cu at (91.7, 31.1)
- added C4: 100n, Capacitor_SMD:C_0603_1608Metric_Pad1.05x0.95mm_HandSolder, F.Cu at (85.3, 30.4)
- added C5: 100n, Capacitor_SMD:C_0603_1608Metric_Pad1.05x0.95mm_HandSolder, F.Cu at (88.7, 27.3)
- added C6: 10n, Capacitor_SMD:C_0603_1608Metric_Pad1.05x0.95mm_HandSolder, F.Cu at (44.9, 37.0)
- added C7: 10n, Capacitor_SMD:C_0603_1608Metric_Pad1.05x0.95mm_HandSolder, F.Cu at (44.9, 35.5)
- added C8: 10n, Capacitor_SMD:C_0603_1608Metric_Pad1.05x0.95mm_HandSolder, F.Cu at (38.8, 45.5)
- added C9: 100n, Capacitor_SMD:C_0603_1608Metric_Pad1.05x0.95mm_HandSolder, F.Cu at (35.4, 47.0)
- added D1: 150060VS75020, LED_SMD:LED_0603_1608Metric_Pad1.05x0.95mm_HandSolder, F.Cu at (74.3, 41.3)
- added D10: 150060AS75000, LED_SMD:LED_0603_1608Metric_Pad1.05x0.95mm_HandSolder, F.Cu at (32.3, 37.2)
- added D11: 150060AS75000, LED_SMD:LED_0603_1608Metric_Pad1.05x0.95mm_HandSolder, F.Cu at (71.7, 56.1)
- added D2: CDSW4448-G, Diode_SMD:D_SOD-123, F.Cu at (35.2, 28.3)
- added D3: CDSW4448-G, Diode_SMD:D_SOD-123, F.Cu at (39.9, 25.9)
- added D4: CDSW4448-G, Diode_SMD:D_SOD-123, F.Cu at (45.6, 33.6)
- added D5: CDSW4448-G, Diode_SMD:D_SOD-123, F.Cu at (35.2, 25.9)
- added D6: BZT52C8V2S-7-F, Diode_SMD:D_SOD-323_HandSoldering, F.Cu at (39.6, 28.1)
- added D7: 150060RS75020, LED_SMD:LED_0603_1608Metric_Pad1.05x0.95mm_HandSolder, F.Cu at (35.4, 44.0)
- added D8: CDSW4448-G, Diode_SMD:D_SOD-123, F.Cu at (54.0, 27.9)
- added D9: CDSW4448-G, Diode_SMD:D_SOD-123, F.Cu at (71.1, 27.9)
- added H1: MountingHole_Pad, MountingHole:MountingHole_3.2mm_M3_Pad_Via, F.Cu at (16.5, 17.8)
- added H2: MountingHole_Pad, MountingHole:MountingHole_3.2mm_M3_Pad_Via, F.Cu at (16.5, 91.4)
- added H3: MountingHole_Pad, MountingHole:MountingHole_3.2mm_M3_Pad_Via, F.Cu at (120.5, 88.9)
- added H4: MountingHole_Pad, MountingHole:MountingHole_3.2mm_M3_Pad_Via, F.Cu at (117.3, 17.8)
- added J1: Screw_Terminal_01x02, Connector_PinHeader_2.54mm:PinHeader_1x02_P2.54mm_Vertical, F.Cu at (39.4, 15.2)
- added J2: Screw_Terminal_01x02, Connector_PinHeader_2.54mm:PinHeader_1x02_P2.54mm_Vertical, F.Cu at (48.9, 15.2)
- added J3: Screw_Terminal_01x12, Connector_PinHeader_2.54mm:PinHeader_1x12_P2.54mm_Vertical, F.Cu at (57.1, 15.2)
- added J4: NUCLEO144ZE-STLINK, Connector_PinHeader_2.54mm:PinHeader_1x05_P2.54mm_Vertical, F.Cu at (106.7, 52.0)
- added JP1: Jumper_3_Bridged12, Connector_PinHeader_2.54mm:PinHeader_1x03_P2.54mm_Vertical, F.Cu at (57.1, 19.1)
- added JP2: Jumper_3_Bridged12, Connector_PinHeader_2.54mm:PinHeader_1x03_P2.54mm_Vertical, F.Cu at (62.2, 19.1)
- added JP3: Jumper_3_Bridged12, Connector_PinHeader_2.54mm:PinHeader_1x03_P2.54mm_Vertical, F.Cu at (67.9, 19.1)
- added L1: CIGT201210UHR47MNE, Capacitor_SMD:C_0805_2012Metric, F.Cu at (63.5, 45.7)
- added Q1: STL76DN4LF7AG, STL76DN4LF7AG:STL76DN4LF7AG, F.Cu at (50.2, 21.6)
- added Q2: STL120N4F6AG, STL120N4F6AG:STL120N4F6AG, F.Cu at (45.7, 52.1)
- added Q3: SSM3K337R, Package_TO_SOT_SMD:SOT-23, F.Cu at (32.0, 45.0)
- added Q4: SIS413DN-T1-GE3, Package_SO:Vishay_PowerPAK_1212-8_Single, F.Cu at (44.1, 44.8)
- added Q5: SSM3K337R, Package_TO_SOT_SMD:SOT-23, F.Cu at (57.1, 27.9)
- added Q6: SSM3K337R, Package_TO_SOT_SMD:SOT-23, F.Cu at (62.2, 27.9)
- added Q7: SSM3K337R, Package_TO_SOT_SMD:SOT-23, F.Cu at (67.9, 27.9)
- added R1: 1k, Resistor_SMD:R_0603_1608Metric_Pad1.05x0.95mm_HandSolder, F.Cu at (66.1, 64.8)
- added R10: 0, Resistor_SMD:R_0603_1608Metric_Pad1.05x0.95mm_HandSolder, F.Cu at (38.7, 47.0)
- added R11: 1k, Resistor_SMD:R_0603_1608Metric_Pad1.05x0.95mm_HandSolder, F.Cu at (44.5, 29.2)
- added R12: 1k, Resistor_SMD:R_0603_1608Metric_Pad1.05x0.95mm_HandSolder, F.Cu at (48.2, 35.5)
- added R13: 1K, Resistor_SMD:R_0603_1608Metric_Pad1.05x0.95mm_HandSolder, F.Cu at (44.9, 38.5)
- added R14: 10k, Resistor_SMD:R_0603_1608Metric_Pad1.05x0.95mm_HandSolder, F.Cu at (48.2, 37.0)
- added R15: 1k, Resistor_SMD:R_0603_1608Metric_Pad1.05x0.95mm_HandSolder, F.Cu at (35.8, 37.5)
- added R16: 1k, Resistor_SMD:R_0603_1608Metric_Pad1.05x0.95mm_HandSolder, F.Cu at (106.7, 30.5)
- added R2: 1k, Resistor_SMD:R_0603_1608Metric_Pad1.05x0.95mm_HandSolder, F.Cu at (66.0, 67.3)
- added R3: 1k, Resistor_SMD:R_0603_1608Metric_Pad1.05x0.95mm_HandSolder, F.Cu at (66.0, 69.8)
- added R4: 1k5, Resistor_SMD:R_0603_1608Metric_Pad1.05x0.95mm_HandSolder, F.Cu at (65.2, 61.7)
- added R5: 10k, Resistor_SMD:R_0603_1608Metric_Pad1.05x0.95mm_HandSolder, F.Cu at (67.1, 61.7)
- added R6: 1k, Resistor_SMD:R_0603_1608Metric_Pad1.05x0.95mm_HandSolder, F.Cu at (110.2, 50.9)
- added R7: 1k, Resistor_SMD:R_0603_1608Metric_Pad1.05x0.95mm_HandSolder, F.Cu at (91.7, 29.3)
- added R8: 10k, Resistor_SMD:R_0603_1608Metric_Pad1.05x0.95mm_HandSolder, F.Cu at (74.3, 39.4)
- added R9: 10k, Resistor_SMD:R_0603_1608Metric_Pad1.05x0.95mm_HandSolder, F.Cu at (38.8, 43.9)
- added SW1: SW, Button_Switch_THT:SW_PUSH_6mm_H5mm, F.Cu at (119.4, 47.0)
- added TP1: TestPoint, Connector_PinHeader_1.27mm:PinHeader_1x01_P1.27mm_Vertical, F.Cu at (84.6, 50.2)
- added TP10: TestPoint, Connector_PinHeader_1.00mm:PinHeader_1x01_P1.00mm_Vertical, F.Cu at (40.0, 40.0)
- added TP11: TestPoint, Connector_PinHeader_1.27mm:PinHeader_1x01_P1.27mm_Vertical, F.Cu at (62.9, 38.1)
- added TP12: TestPoint, Connector_PinHeader_1.27mm:PinHeader_1x01_P1.27mm_Vertical, F.Cu at (62.9, 35.6)
- added TP2: TestPoint, Connector_PinHeader_1.27mm:PinHeader_1x01_P1.27mm_Vertical, F.Cu at (84.6, 47.6)
- added TP3: TestPoint, Connector_PinHeader_1.27mm:PinHeader_1x01_P1.27mm_Vertical, F.Cu at (84.6, 45.0)
- added TP4: TestPoint, Connector_PinHeader_1.27mm:PinHeader_1x01_P1.27mm_Vertical, F.Cu at (84.6, 42.5)
- added TP5: TestPoint, Connector_PinHeader_1.27mm:PinHeader_1x01_P1.27mm_Vertical, F.Cu at (84.6, 40.0)
- added TP6: TestPoint, Connector_PinHeader_1.27mm:PinHeader_1x01_P1.27mm_Vertical, F.Cu at (84.6, 37.5)
- added TP7: TestPoint, Connector_PinHeader_1.27mm:PinHeader_1x01_P1.27mm_Vertical, F.Cu at (44.8, 40.4)
- added TP8: TestPoint, Connector_PinHeader_1.27mm:PinHeader_1x01_P1.27mm_Vertical, F.Cu at (48.1, 38.9)
- added TP9: TestPoint, Connector_PinHeader_1.00mm:PinHeader_1x01_P1.00mm_Vertical, F.Cu at (48.0, 41.1)
- added U1: STM32L031F4Px, Package_SO:TSSOP-20_4.4x6.5mm_P0.65mm, F.Cu at (94.0, 35.6)
- added U2: VNHD7008AY, Package_SO:ST_PowerSSO-36_SlugDown_ThermalVias, F.Cu at (43.2, 61.0)
- added U3: AZ1117IH-3.3TRG1, Package_TO_SOT_SMD:SOT-223-3_TabPin2, F.Cu at (73.7, 49.5)
- added U4: MMA8452Q, Package_DFN_QFN:QFN-16-1EP_3x3mm_P0.5mm_EP1.8x1.8mm, F.Cu at (104.1, 34.3)
Routing:
- added copper zone on F.Cu, net +12V
- added copper zone on F.Cu, net +3V3
- added copper zone on B.Cu, net GND
Other:
- board outline added: 115.6 x 82.5 mm
