File: hw/saber/saber.kicad_pcb (KiCad board)
At the start: 4 copper layers, 60.7 x 27.2 mm, 73 parts, among them J1 282834-2, J2 282834-2, J3 OSTVN12A150, J4 NUCLEO144ZE-STLINK, Q1 STL120N4F6AG, Q2 SIS413DN-T1-GE3, Q3 SSM3K337R, Q4 STL76DN4LF7AG, Q5 SSM3K337R, Q6 SSM3K337R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

Commit message: Initial routing complete
Parts:
- moved R5 3.12 mm to (151.4, 86.5)
- moved R4 1.55 mm to (152.9, 86.5)
- moved C1 1.54 mm to (154.5, 86.5), turned to 270 degrees
- moved R7 1.04 mm to (172.2, 82.5)
- moved R20 1.01 mm to (171.4, 73.5)
- moved SW1 0.84 mm to (173.2, 76.5)
- moved R14 0.63 mm to (143.5, 67.4)
- moved R15 0.63 mm to (144.8, 67.4)
- moved C7 0.51 mm to (125.9, 77.5)
- moved C6 0.25 mm to (121.9, 83.8)
- moved C16 0.11 mm to (175.7, 76.3)
- moved D12 0.11 mm to (146.4, 69.7)
Connections:
- C2 pad 1: +3V3 -> /micro/NRST
- J4 pad 5: +3V3 -> /micro/NRST
- R7 pad 1: Net-(R7-Pad1) -> +3V3
- R7 pad 2: GND -> /micro/NRST
- SW1 pad 1: +3V3 -> /micro/NRST
- SW1 pad 2: Net-(R7-Pad1) -> GND
- U1 pad 13: Net-(U1-Pad13) -> /micro/LED_HBEAT
- U1 pad 14: Net-(U1-Pad14) -> /actuators/SIG_SOL
- U1 pad 15: Net-(U1-Pad15) -> /actuators/SIG_LED
- U1 pad 18: /actuators/SIG_SOL -> Net-(U1-Pad18)
- U1 pad 19: /actuators/SIG_LED -> /BTN
- U1 pad 4: +3V3 -> /micro/NRST
- U1 pad 8: Net-(U1-Pad8) -> /actuators/PWM_SPKR
Routing:
- net GND: track 83.2 -> 107.8 mm, vias 29 -> 36
- net /acc/SDA: track 5.96 -> 29.9 mm
- net /micro/NRST: track 0.00 -> 19.7 mm, vias 0 -> 1
- net /micro/INB_MCU: track 0.00 -> 17.4 mm
- net /micro/PWM_MTR_MCU: track 0.00 -> 15.3 mm
- net /actuators/SIG_SOL: track 1.19 -> 14.8 mm, vias 1 -> 0
- net /actuators/PWM_SPKR: track 1.19 -> 14.0 mm, vias 1 -> 0
- net +12V: track 2.20 -> 12.6 mm, vias 4 -> 6
- net /LED+: track 3.77 -> 13.5 mm
- net +3V3: track 35.3 -> 44.5 mm, vias 11 -> 18
- net /SPKR+: track 3.81 -> 12.4 mm
- net /ENC_A: track 1.97 -> 10.4 mm
- net /micro/ADC_imtr: track 0.00 -> 8.44 mm
- net /actuators/SIG_LED: track 1.19 -> 9.52 mm, vias 1 -> 0
- net /ENC_B: track 2.98 -> 11.1 mm
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